File: audrey-ii-simple_electronics/AudioBufferOut.kicad_sch (KiCad schematic)
At the start: 17 parts, among them J1 DAC_OUT_2, J2 DAC_OUT_2, U1 TL074

Commit message: -
Parts:
- added C9: 100n, Capacitor_SMD:C_0603_1608Metric, symbol Device:C_Small
- C1, C2, C3, C4: LCSC# (none) -> C1671
- R1, R2: LCSC# (none) -> C25804
- R10, R9: LCSC# (none) -> C21190
- R3, R4, R5, R6, R7, R8: LCSC# (none) -> C25803
- U1: LCSC# (none) -> C6964
Connections:
- net AUDIO_OUT_L: no longer J1.T, R9.2
- net AUDIO_OUT_R: no longer J2.T, R10.2
- net GND: now also U1.4 (V+), C9.2
- net +3.3VA: now reaches U1.11 (V-)
- net +3.3VA: now also C9.1
- new net: J1.T, R9.2
- new net: J2.T, R10.2
Other:
- moved on the sheet: U1E
