File: audrey-ii-simple_electronics/GPIOIn.kicad_sch (KiCad schematic)
At the start: 6 parts, among them J1 DAC_OUT_2, Q1 MMBT3904

Commit message: -
Parts:
- Q1: LCSC# (none) -> C20526
- R60: LCSC# (none) -> C25803
- R61: LCSC# (none) -> C136593
- R62: LCSC# (none) -> C25804
- R63: LCSC# (none) -> C21190
Changed lines of the file:
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@@
+      (effects (font (size 1.27 1.27)) hide)
+    )
+    (property "LCSC#" "C25804" (at 130.81 80.01 0)
       (effects (font (size 1.27 1.27)) hide)
     )
@@
       (effects (font (size 1.27 1.27)) hide)
     )
+    (property "LCSC#" "C21190" (at 140.97 86.36 0)
+      (effects (font (size 1.27 1.27)) hide)
+    )
     (pin "1")
     (pin "2")
@@
       (effects (font (size 1.27 1.27)) hide)
     )
+    (property "LCSC#" "C25803" (at 114.3 95.25 0)
+      (effects (font (size 1.27 1.27)) hide)
+    )
     (pin "1")
     (pin "2")
@@
     )
     (property "Datasheet" "~" (at 120.65 105.41 0)
+      (effects (font (size 1.27 1.27)) hide)
+    )
+    (property "LCSC#" "C136593" (at 120.65 105.41 0)
       (effects (font (size 1.27 1.27)) hide)
     )
@@
       (effects (font (size 1.27 1.27)) (justify left) hide)
     )
+    (property "LCSC#" "C20526" (at 128.27 95.25 0)
+      (effects (font (size 1.27 1.27)) hide)
+    )
     (pin "1")
