File: audrey-ii-simple_electronics/audrey-ii-simple_electronics.kicad_sch (KiCad schematic)
At the start: 2 parts

Commit message: -
Parts:
- removed U$1: OLED128X64, Connector_PinSocket_2.54mm:PinSocket_1x20_P2.54mm_Vertical, symbol teletype_clone-eagle-import:OLED128X64
Other:
- note removed: "Jumper Option #1 - Independent Supply Voltage for Boost Converter (BC_VDD) R4 R5 R7 Description Open Close Open Boost converter + OLED panel are powered from BC_VDD (pin #3). OLED controller is still powered from VDD (pin #2). This allows for increased efficiency through the boost converter, by allowing a supply voltage up to +12V at its input, BC_VDD (pin #3)"
- note removed: "REMEMBER TO CONFIGURE THE RESISTORS AS DESCRIBED IN THE DATASHEET"
- note removed: "https://www.mouser.dk/datasheet/2/291/NHD_2_7_12864WDY3-2952904.pdf PAGE 5"
