File: audrey-ii-simple_electronics/ADCBufferIn.kicad_sch (KiCad schematic)
At the start: 30 parts, among them J3 CV_1, J4 CV_2, J5 CV_3, J6 CV_4, U2 MCP6004

Commit message: -
Parts:
- C5, C6, C7, C8: LCSC# (none) -> C57112
- C9: LCSC# (none) -> C14663
- R11, R13, R14, R16, R17, R19, R20, R22, R23, R24, R25, R26: LCSC# (none) -> C403321
- R12, R15, R18, R21: LCSC# (none) -> C25803
- U2: LCSC# (none) -> C7378
Changed lines of the file:
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@@
+      (effects (font (size 1.27 1.27)) hide)
+    )
+    (property "LCSC#" "C25803" (at 55.88 184.15 0)
       (effects (font (size 1.27 1.27)) hide)
     )
@@
       (effects (font (size 1.27 1.27)) hide)
     )
+    (property "LCSC#" "C14663" (at 166.37 172.72 0)
+      (effects (font (size 1.27 1.27)) hide)
+    )
     (pin "1")
     (pin "2")
@@
       (effects (font (size 1.27 1.27)) hide)
     )
+    (property "LCSC#" "C57112" (at 83.82 154.94 0)
+      (effects (font (size 1.27 1.27)) hide)
+    )
     (pin "1")
     (pin "2")
@@
       (effects (font (size 1.27 1.27)) hide)
     )
+    (property "LCSC#" "C403321" (at 55.88 129.54 0)
+      (effects (font (size 1.27 1.27)) hide)
+    )
     (pin "1")
     (pin "2")
@@
       (effects (font (size 1.27 1.27)) hide)
     )
+    (property "LCSC#" "C403321" (at 55.88 100.33 0)
+      (effects (font (size 1.27 1.27)) hide)
+    )
     (pin "1")
     (pin "2")
@@
     )
     (property "Datasheet" "http://ww1.microchip.com/downloads/en/DeviceDoc/21733j.pdf" (at 86.36 49.53 0)
+      (effects (font (size 1.27 1.27)) hide)
+    )
+    (property "LCSC#" "C7378" (at 85.09 44.45 0)
       (effects (font (size 1.27 1.27)) hide)
     )
@@
       (effects (font (size 1.27 1.27)) hide)
     )
+    (property "LCSC#" "C25803" (at 55.88 137.16 0)
+      (effects (font (size 1.27 1.27)) hide)
+    )
     (pin "1")
     (pin "2")
@@
     )
     (property "Datasheet" "~" (at 55.88 57.15 0)
+      (effects (font (size 1.27 1.27)) hide)
+    )
+    (property "LCSC#" "C403321" (at 55.88 57.15 0)
       (effects (font (size 1.27 1.27)) hide)
     )
@@
       (effects (font (size 1.27 1.27)) hide)
     )
+    (property "LCSC#" "C403321" (at 83.82 73.66 0)
+      (effects (font (size 1.27 1.27)) hide)
+    )
     (pin "1")
     (pin "2")
@@
       (effects (font (size 1.27 1.27)) hide)
     )
+    (property "LCSC#" "C25803" (at 55.88 49.53 0)
+      (effects (font (size 1.27 1.27)) hide)
+    )
     (pin "1")
     (pin "2")
@@
       (effects (font (size 1.27 1.27)) hide)
     )
+    (property "LCSC#" "C25803" (at 55.88 92.71 0)
+      (effects (font (size 1.27 1.27)) hide)
+    )
     (pin "1")
     (pin "2")
@@
     )
     (property "Datasheet" "http://ww1.microchip.com/downloads/en/DeviceDoc/21733j.pdf" (at 86.36 184.15 0)
+      (effects (font (size 1.27 1.27)) hide)
+    )
+    (property "LCSC#" "C7378" (at 85.09 179.07 0)
       (effects (font (size 1.27 1.27)) hide)
     )
@@
       (effects (font (size 1.27 1.27)) hide)
     )
+    (property "LCSC#" "C7378" (at 161.29 175.26 0)
+      (effects (font (size 1.27 1.27)) hide)
+    )
     (pin "1")
     (pin "2")
@@
       (effects (font (size 1.27 1.27)) hide)
     )
+    (property "LCSC#" "C403321" (at 55.88 85.09 0)
+      (effects (font (size 1.27 1.27)) hide)
+    )
     (pin "1")
     (pin "2")
@@
     )
     (property "Datasheet" "http://ww1.microchip.com/downloads/en/DeviceDoc/21733j.pdf" (at 86.36 92.71 0)
+      (effects (font (size 1.27 1.27)) hide)
+    )
+    (property "LCSC#" "C7378" (at 85.09 87.63 0)
       (effects (font (size 1.27 1.27)) hide)
     )
@@
       (effects (font (size 1.27 1.27)) hide)
     )
+    (property "LCSC#" "C57112" (at 83.82 107.95 0)
+      (effects (font (size 1.27 1.27)) hide)
+    )
     (pin "1")
     (pin "2")
@@
       (effects (font (size 1.27 1.27)) hide)
     )
+    (property "LCSC#" "C57112" (at 83.82 20.32 0)
+      (effects (font (size 1.27 1.27)) hide)
+    )
     (pin "1")
     (pin "2")
@@
       (effects (font (size 1.27 1.27)) hide)
     )
+    (property "LCSC#" "C57112" (at 83.82 63.5 0)
+      (effects (font (size 1.27 1.27)) hide)
+    )
     (pin "1")
     (pin "2")
@@
     )
     (property "Datasheet" "~" (at 55.88 176.53 0)
+      (effects (font (size 1.27 1.27)) hide)
+    )
+    (property "LCSC#" "C403321" (at 55.88 176.53 0)
       (effects (font (size 1.27 1.27)) hide)
     )
@@
       (effects (font (size 1.27 1.27)) hide)
     )
+    (property "LCSC#" "C403321" (at 83.82 165.1 0)
+      (effects (font (size 1.27 1.27)) hide)
+    )
     (pin "1")
     (pin "2")
@@
       (effects (font (size 1.27 1.27)) hide)
     )
+    (property "LCSC#" "C403321" (at 83.82 30.48 0)
+      (effects (font (size 1.27 1.27)) hide)
+    )
     (pin "1")
     (pin "2")
@@
       (effects (font (size 1.27 1.27)) hide)
     )
+    (property "LCSC#" "C403321" (at 55.88 41.91 0)
+      (effects (font (size 1.27 1.27)) hide)
+    )
     (pin "1")
     (pin "2")
@@
     )
     (property "Datasheet" "http://ww1.microchip.com/downloads/en/DeviceDoc/21733j.pdf" (at 86.36 137.16 0)
+      (effects (font (size 1.27 1.27)) hide)
+    )
+    (property "LCSC#" "C7378" (at 85.09 132.08 0)
       (effects (font (size 1.27 1.27)) hide)
     )
@@
       (effects (font (size 1.27 1.27)) hide)
     )
+    (property "LCSC#" "C403321" (at 83.82 118.11 0)
+      (effects (font (size 1.27 1.27)) hide)
+    )
     (pin "1")
     (pin "2")
@@
       (effects (font (size 1.27 1.27)) hide)
     )
+    (property "LCSC#" "C403321" (at 55.88 191.77 0)
+      (effects (font (size 1.27 1.27)) hide)
+    )
     (pin "1")
     (pin "2")
@@
       (effects (font (size 1.27 1.27)) hide)
     )
+    (property "LCSC#" "C403321" (at 55.88 144.78 0)
+      (effects (font (size 1.27 1.27)) hide)
+    )

Commit message: -
Connections:
- net GND: now also J3.S, J4.S, J5.S, J6.S
Changed lines of the file:
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@@
+    (stroke (width 0) (type default))
+  )
+  (wire (pts (xy 33.02 186.69) (xy 35.56 186.69))
     (stroke (width 0) (type default))
   )
@@
     (stroke (width 0) (type default))
   )
+  (wire (pts (xy 33.02 139.7) (xy 35.56 139.7))
+    (stroke (width 0) (type default))
+  )
   (wire (pts (xy 189.23 52.07) (xy 189.23 54.61))
     (stroke (width 0) (type default))
@@
     (stroke (width 0) (type default))
   )
+  (wire (pts (xy 33.02 95.25) (xy 35.56 95.25))
+    (stroke (width 0) (type default))
+  )
   (wire (pts (xy 189.23 39.37) (xy 203.2 39.37))
     (stroke (width 0) (type default))
@@
     (stroke (width 0) (type default))
   )
+  (wire (pts (xy 35.56 95.25) (xy 35.56 97.79))
+    (stroke (width 0) (type default))
+  )
   (wire (pts (xy 33.02 49.53) (xy 53.34 49.53))
     (stroke (width 0) (type default))
@@
     (stroke (width 0) (type default))
   )
+  (wire (pts (xy 35.56 186.69) (xy 35.56 189.23))
+    (stroke (width 0) (type default))
+  )
   (wire (pts (xy 58.42 137.16) (xy 63.5 137.16))
     (stroke (width 0) (type default))
@@
     (stroke (width 0) (type default))
   )
+  (wire (pts (xy 35.56 139.7) (xy 35.56 142.24))
+    (stroke (width 0) (type default))
+  )
   (wire (pts (xy 81.28 30.48) (xy 72.39 30.48))
     (stroke (width 0) (type default))
@@
     (stroke (width 0) (type default))
   )
+  (wire (pts (xy 33.02 52.07) (xy 35.56 52.07))
+    (stroke (width 0) (type default))
+  )
   (wire (pts (xy 166.37 184.15) (xy 166.37 175.26))
     (stroke (width 0) (type default))
@@
   )
   (wire (pts (xy 72.39 134.62) (xy 77.47 134.62))
+    (stroke (width 0) (type default))
+  )
+  (wire (pts (xy 35.56 52.07) (xy 35.56 54.61))
     (stroke (width 0) (type default))
   )
@@
         (path "/6f2c1bc8-f9c2-4b61-b9a9-e89205eec081/e4ceba68-83be-4e50-b9c0-040298eeacff"
           (reference "R27") (unit 1)
+        )
+      )
+    )
+  )
+  (symbol (lib_id "power:GND") (at 35.56 142.24 0) (unit 1)
+    (in_bom yes) (on_board yes) (dnp no) (fields_autoplaced)
+    (property "Reference" "#PWR058" (at 35.56 148.59 0)
+      (effects (font (size 1.27 1.27)) hide)
+    )
+    (property "Value" "GND" (at 35.56 146.3755 0)
+      (effects (font (size 1.27 1.27)))
+    )
+    (property "Footprint" "" (at 35.56 142.24 0)
+      (effects (font (size 1.27 1.27)) hide)
+    )
+    (property "Datasheet" "" (at 35.56 142.24 0)
+      (effects (font (size 1.27 1.27)) hide)
+    )
+    (pin "1")
+    (instances
+      (project "audrey-ii-simple_electronics"
+        (path "/655d86ff-20fd-40aa-a4fb-11d32a0c01aa/19f795e2-a875-4961-aba5-130ac500cd0c"
+          (reference "#PWR058") (unit 1)
+        )
+        (path "/655d86ff-20fd-40aa-a4fb-11d32a0c01aa/009d8bc5-9444-4666-8502-b88a2706b3ff"
+          (reference "#PWR059") (unit 1)
+        )
+        (path "/655d86ff-20fd-40aa-a4fb-11d32a0c01aa/42aaa187-b73e-4283-8802-9e8dd9842439"
+          (reference "#PWR060") (unit 1)
+        )
+      )
+      (project "daisy_dev"
+        (path "/6f2c1bc8-f9c2-4b61-b9a9-e89205eec081/e4ceba68-83be-4e50-b9c0-040298eeacff"
+          (reference "#PWR018") (unit 1)
         )
       )
@@
     )
   )
+  (symbol (lib_id "power:GND") (at 35.56 97.79 0) (unit 1)
+    (in_bom yes) (on_board yes) (dnp no) (fields_autoplaced)
+    (property "Reference" "#PWR055" (at 35.56 104.14 0)
+      (effects (font (size 1.27 1.27)) hide)
+    )
+    (property "Value" "GND" (at 35.56 101.9255 0)
+      (effects (font (size 1.27 1.27)))
+    )
+    (property "Footprint" "" (at 35.56 97.79 0)
+      (effects (font (size 1.27 1.27)) hide)
+    )
+    (property "Datasheet" "" (at 35.56 97.79 0)
+      (effects (font (size 1.27 1.27)) hide)
+    )
+    (pin "1")
+    (instances
+      (project "audrey-ii-simple_electronics"
+        (path "/655d86ff-20fd-40aa-a4fb-11d32a0c01aa/19f795e2-a875-4961-aba5-130ac500cd0c"
+          (reference "#PWR055") (unit 1)
+        )
+        (path "/655d86ff-20fd-40aa-a4fb-11d32a0c01aa/009d8bc5-9444-4666-8502-b88a2706b3ff"
+          (reference "#PWR056") (unit 1)
+        )
+        (path "/655d86ff-20fd-40aa-a4fb-11d32a0c01aa/42aaa187-b73e-4283-8802-9e8dd9842439"
+          (reference "#PWR057") (unit 1)
+        )
+      )
+      (project "daisy_dev"
+        (path "/6f2c1bc8-f9c2-4b61-b9a9-e89205eec081/e4ceba68-83be-4e50-b9c0-040298eeacff"
+          (reference "#PWR018") (unit 1)
+        )
+      )
+    )
+  )
   (symbol (lib_id "Device:R_Potentiometer_Small") (at 231.14 45.72 0) (unit 1)
     (in_bom yes) (on_board yes) (dnp no) (fields_autoplaced)
@@
     )
   )
+  (symbol (lib_id "power:GND") (at 35.56 54.61 0) (unit 1)
+    (in_bom yes) (on_board yes) (dnp no) (fields_autoplaced)
+    (property "Reference" "#PWR044" (at 35.56 60.96 0)
+      (effects (font (size 1.27 1.27)) hide)
+    )
+    (property "Value" "GND" (at 35.56 58.7455 0)
+      (effects (font (size 1.27 1.27)))
+    )
+    (property "Footprint" "" (at 35.56 54.61 0)
+      (effects (font (size 1.27 1.27)) hide)
+    )
+    (property "Datasheet" "" (at 35.56 54.61 0)
+      (effects (font (size 1.27 1.27)) hide)
+    )
+    (pin "1")
+    (instances
+      (project "audrey-ii-simple_electronics"
+        (path "/655d86ff-20fd-40aa-a4fb-11d32a0c01aa/19f795e2-a875-4961-aba5-130ac500cd0c"
+          (reference "#PWR044") (unit 1)
+        )
+        (path "/655d86ff-20fd-40aa-a4fb-11d32a0c01aa/009d8bc5-9444-4666-8502-b88a2706b3ff"
+          (reference "#PWR045") (unit 1)
+        )
+        (path "/655d86ff-20fd-40aa-a4fb-11d32a0c01aa/42aaa187-b73e-4283-8802-9e8dd9842439"
+          (reference "#PWR046") (unit 1)
+        )
+      )
+      (project "daisy_dev"
+        (path "/6f2c1bc8-f9c2-4b61-b9a9-e89205eec081/e4ceba68-83be-4e50-b9c0-040298eeacff"
+          (reference "#PWR018") (unit 1)
+        )
+      )
+    )
+  )
   (symbol (lib_id "Connector_Audio:AudioJack2_SwitchT") (at 27.94 184.15 0) (mirror x) (unit 1)
     (in_bom yes) (on_board yes) (dnp no)
@@
         )
       )
+    )
+  )
+  (symbol (lib_id "power:GND") (at 35.56 189.23 0) (unit 1)
+    (in_bom yes) (on_board yes) (dnp no) (fields_autoplaced)
+    (property "Reference" "#PWR061" (at 35.56 195.58 0)
+      (effects (font (size 1.27 1.27)) hide)
+    )
+    (property "Value" "GND" (at 35.56 193.3655 0)
+      (effects (font (size 1.27 1.27)))
+    )
+    (property "Footprint" "" (at 35.56 189.23 0)
+      (effects (font (size 1.27 1.27)) hide)
+    )
+    (property "Datasheet" "" (at 35.56 189.23 0)
+      (effects (font (size 1.27 1.27)) hide)
+    )
+    (pin "1")
+    (instances
+      (project "audrey-ii-simple_electronics"
+        (path "/655d86ff-20fd-40aa-a4fb-11d32a0c01aa/19f795e2-a875-4961-aba5-130ac500cd0c"
+          (reference "#PWR061") (unit 1)
+        )
+        (path "/655d86ff-20fd-40aa-a4fb-11d32a0c01aa/009d8bc5-9444-4666-8502-b88a2706b3ff"
+          (reference "#PWR062") (unit 1)
+        )
+        (path "/655d86ff-20fd-40aa-a4fb-11d32a0c01aa/42aaa187-b73e-4283-8802-9e8dd9842439"
+          (reference "#PWR063") (unit 1)
+        )
+      )
+      (project "daisy_dev"
+        (path "/6f2c1bc8-f9c2-4b61-b9a9-e89205eec081/e4ceba68-83be-4e50-b9c0-040298eeacff"
+          (reference "#PWR018") (unit 1)
+        )
+      )
