File: audrey-ii-simple_electronics/SPDT.kicad_sch (KiCad schematic)
At the start: 2 parts, among them SW1 SW_SPDT

Commit message: -
Parts:
- R63: LCSC# (none) -> C21190
Changed lines of the file:
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@@
+      (effects (font (size 1.27 1.27)) hide)
+    )
+    (property "LCSC#" "C21190" (at 151.13 85.09 0)
       (effects (font (size 1.27 1.27)) hide)
     )

Commit message: -
Parts:
- SW1: footprint (none) -> Connector_PinHeader_2.54mm:PinHeader_1x03_P2.54mm_Vertical
Changed lines of the file:
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@@
       (effects (font (size 1.27 1.27)))
     )
-    (property "Footprint" "" (at 138.43 97.79 0)
+    (property "Footprint" "Connector_PinHeader_2.54mm:PinHeader_1x03_P2.54mm_Vertical" (at 138.43 97.79 0)
       (effects (font (size 1.27 1.27)) hide)
     )
