File: audrey-ii-simple_electronics/audrey-ii-simple_electronics.kicad_pcb (KiCad board)
At the start: 2 copper layers, 172.7 x 128.5 mm, 125 parts, among them J1 DAC_OUT_2, J10 CV_4, J11 CV_1, J12 CV_2, J13 CV_3, J14 CV_4, J15 Conn_02x05_Odd_Even, J16 DAC_OUT_2, J2 DAC_OUT_2, J3 CV_1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

Commit message: -
Parts:
- removed U$1: OLED128X64, Connector_PinSocket_2.54mm:PinSocket_1x20_P2.54mm_Vertical
- added C23: 100n, Capacitor_SMD:C_0603_1608Metric, F.Cu at (86.6, 133.6)
- added C24: 10uF, Capacitor_Tantalum_SMD:CP_EIA-3216-18_Kemet-A, F.Cu at (82.5, 133.1)
- added C25: 100n, Capacitor_SMD:C_0603_1608Metric, F.Cu at (200.9, 135.6)
- D1, D2: footprint Diode_SMD:D_SOD-123 -> Diode_SMD:D_SMA
- U5: value LM4040DCK-2.0 -> LM4040-10V; footprint Package_TO_SOT_SMD:SOT-353_SC-70-5 -> Package_TO_SOT_SMD:SOT-23-3
- moved Q1 127.0 mm to (235.5, 108.0), turned to 180 degrees
- moved J16 125.5 mm to (235.7, 119.4)
- moved R61 124.8 mm to (239.0, 109.0), turned to 180 degrees
- moved R60 124.4 mm to (239.0, 107.3), turned to 180 degrees
- moved R62 122.3 mm to (232.7, 106.7), turned to 90 degrees
- moved R63 121.8 mm to (231.9, 109.0)
- moved R64 118.0 mm to (214.4, 116.8)
- moved C22 33.2 mm to (105.7, 124.7), turned to -90 degrees
- moved R59 28.8 mm to (103.6, 124.7), turned to -90 degrees
- moved R6 27.0 mm to (198.5, 132.1), turned to -90 degrees
- moved R8 26.9 mm to (200.1, 138.9), turned to -90 degrees
- moved C4 24.9 mm to (201.7, 138.9), turned to 90 degrees
- moved R4 24.4 mm to (200.3, 132.1), turned to 90 degrees
- moved R10 23.6 mm to (204.2, 143.2), turned to -90 degrees
- moved C2 22.0 mm to (202.0, 132.2), turned to -90 degrees
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Connections:
- J15 pad 9: unconnected-(J15-Pin_9-Pad9) -> Net-(D1-A)
- U1 pad 11: unconnected-(U1E-V--Pad11) -> +3.3VA
- U1 pad 4: unconnected-(U1E-V+-Pad4) -> GND
- U5 pad 1: -10V_REF -> GND
- U5 pad 2: (no net) -> -10V_REF
- U5 pad 3: GND -> (no net)
Routing:
- net /ADCBufferIn/ADC_4: track 0.00 -> 75.7 mm, vias 0 -> 1
- net /ADCBufferIn/KNOB_2: track 0.00 -> 73.0 mm
- net /ADCBufferIn/ADC_1: track 0.00 -> 69.9 mm, vias 0 -> 1
- net /ADCBufferIn/ADC_2: track 0.00 -> 61.0 mm, vias 0 -> 1
- net -10V_REF: track 0.00 -> 58.5 mm
- net /ADCBufferIn/KNOB_1: track 0.00 -> 54.4 mm
- net Net-(J3-PadT): track 0.00 -> 23.8 mm
- net VEE: track 0.00 -> 17.1 mm
- net Net-(U2D--): track 0.00 -> 16.6 mm
- net Net-(U2C--): track 0.00 -> 15.1 mm
- net Net-(U2A--): track 0.00 -> 14.4 mm
- net Net-(U2B--): track 0.00 -> 14.1 mm
- net VCC: track 0.00 -> 13.7 mm
- net Net-(D1-A): track 0.00 -> 10.8 mm
- net +5V: track 0.00 -> 8.95 mm
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- added copper zone on B.Cu, net GND
- added copper zone on F.Cu, net GND
Other:
- board size 172.7 x 128.5 mm -> 342.6 x 128.5 mm
- board text added: "body"
- board text added: "delay time"
- board text added: "dry/wet"
- board text added: "frequency"
- board text added: "highpass"
- board text added: "lowpass"
- board text added: "misc"
- board text added: "mix"
- board text added: "repeats"
- board text added: "reverb"
- board text added: "volumen"

Commit message: -
Parts:
- added SW1: SW_SPDT, Connector_PinHeader_2.54mm:PinHeader_1x03_P2.54mm_Vertical, F.Cu at (216.4, 115.1)
- moved R54 50.5 mm to (184.0, 97.0), turned to 180 degrees
- moved R52 48.9 mm to (184.0, 98.6), turned to 180 degrees
- moved R58 45.8 mm to (179.8, 97.8), turned to 90 degrees
- moved R53 45.0 mm to (173.6, 94.5), turned to -90 degrees
- moved C18 44.4 mm to (178.2, 97.8), turned to -90 degrees
- moved R44 44.0 mm to (171.9, 94.5), turned to -90 degrees
- moved R49 43.9 mm to (183.9, 103.8), turned to 180 degrees
- moved R51 42.4 mm to (183.9, 105.5), turned to 180 degrees
- moved R57 38.6 mm to (179.9, 104.8), turned to -90 degrees
- moved C17 37.0 mm to (178.3, 104.8), turned to 90 degrees
- moved C15 36.2 mm to (166.8, 98.5), turned to -90 degrees
- moved R45 35.9 mm to (161.6, 97.8), turned to 0 degrees
- moved R55 35.7 mm to (165.2, 98.5), turned to 90 degrees
- moved U4 35.6 mm to (172.5, 101.5), turned to 0 degrees
- moved R43 33.6 mm to (161.6, 99.4), turned to 0 degrees
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Connections:
- J10 pad S: unconnected-(J10-PadS) -> GND
- J11 pad S: unconnected-(J11-PadS) -> GND
- J12 pad S: unconnected-(J12-PadS) -> GND
- J13 pad S: unconnected-(J13-PadS) -> GND
- J14 pad S: unconnected-(J14-PadS) -> GND
- J3 pad S: unconnected-(J3-PadS) -> GND
- J4 pad S: unconnected-(J4-PadS) -> GND
- J5 pad S: unconnected-(J5-PadS) -> GND
- J6 pad S: unconnected-(J6-PadS) -> GND
- J7 pad S: unconnected-(J7-PadS) -> GND
- J8 pad S: unconnected-(J8-PadS) -> GND
- J9 pad S: unconnected-(J9-PadS) -> GND
Routing:
- net -10V_REF: track 58.5 -> 199.4 mm, vias 0 -> 9
- net Net-(J10-PadT): track 0.00 -> 129.3 mm, vias 0 -> 1
- net /ADCBufferIn1/KNOB_4: track 0.00 -> 125.6 mm, vias 0 -> 1
- net /ADCBufferIn2/KNOB_2: track 0.00 -> 114.0 mm, vias 0 -> 1
- net /ADCBufferIn/KNOB_4: track 0.00 -> 95.1 mm, vias 0 -> 1
- net /SPDT/I/O: track 0.00 -> 87.7 mm, vias 0 -> 1
- net Net-(J6-PadT): track 0.00 -> 82.0 mm, vias 0 -> 1
- net Net-(J13-PadT): track 0.00 -> 81.8 mm, vias 0 -> 1
- net /Audio Buffer Out/AUDIO_OUT_R: track 0.00 -> 81.1 mm
- net /GPIOIn/In: track 0.00 -> 80.1 mm, vias 0 -> 1
- net /Audio Buffer Out/AUDIO_OUT_L: track 0.00 -> 71.8 mm, vias 0 -> 2
- net /ADCBufferIn1/KNOB_2: track 0.00 -> 71.4 mm, vias 0 -> 2
- net /ADCBufferIn/ADC_3: track 5.08 -> 72.2 mm, vias 0 -> 1
- net Net-(J12-PadT): track 0.00 -> 67.1 mm, vias 0 -> 1
- net /ADCBufferIn1/KNOB_3: track 0.00 -> 65.1 mm, vias 0 -> 2
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- added copper zone on In2.Cu, net +3.3VA
Other:
- copper layers 2 -> 4
- board text added: "volume"
- board text removed: "volumen"

Commit message: front panel
Other:
- board size 342.6 x 128.5 mm -> 353.6 x 128.5 mm
- board text added: "DELAY SWITCH"
- board text added: "DELAY TIME"
- board text added: "FREQUENCY"
- board text added: "LEFT OUT"
- board text added: "MIX"
- board text added: "RIGHT OUT"
- board text added: "VOLUME"
